File: schematics/rev2/ScouseTom_CS_Shield.sch (EAGLE design)
At the start: 101 parts, among them IC1 REG1117, IC2 REG1117, IC3 OPA2188AID, U1 AD9954YSVZ, U2 LTC69000, U6 LTC1044CS8PBF, U7 ADUM240D0BRIZ, U8 ADUM240D0BRIZ

Commit message: board finished
Parts:
- added JP2, JP4: (no value), pinhead:PINHD-1X2
- renumbered R1_0.1% to R1_H, R1_DAC_1% to R1_DAC, R2_0.1% to R2_H, R2_DAC_1% to R2_DAC, R3_DAC_1% to R3_DAC, R4_DAC_1% to R4_DAC, R6_0.1% to R6_H, R7_0.1% to R7_H, RF_DAC_1% to RF_DAC, RG_DAC_1% to RG_DAC, RX_DAC_1% to RX_DAC, RY_DAC_1% to RY_DAC, R_GAIN1_0.1% to R_HG1, R_GAIN2_0.1% to R_HG2, R_GAIN3_0.1% to R_HG3, R_SET1_0.1% to R_SET1
Connections:
- net GND: now also JP2.2, JP4.1, U$2.GND@5
- net VBAT+: now also JP2.1
- net VBAT-: now also JP4.2
Other:
- note added: "backup THD ones"
- moved on the sheet: DSUB3, JP5

Commit message: Latest Rev2 and USB_ISO
Parts:
- C13, C15, C16, C17, C19, C20, C24, C25, C29, C30, C32, C33: device resistor:C-EUC0805 -> resistor:C-EUC0603
- IC3: value OPA2188AID -> OPA2188AIDGKR; device OPA2188AID:OPA2188AID -> OPA2188AIDGKR:OPA2188AIDGKR
- U2: value LTC69000 -> LTC6900_LTC69000; device LTC6900:LTC69000 -> Low.Noise.Current.Source:LTC6900_LTC69000
Other:
- note added: "Iout=Vin/RG"
- note added: "Set output current by connecting jumper to appropriate resistor: 2k: 250uA 5k: 100uA 10k: 50uA"
- note added: "Vin is 0.5V from DAC"
- note removed: "Set output current by connecting jumper to appropriate resistor: 2k: 500uA 5k: 200uA 10k: 100uA"
